Commit message: Got action and joint trajectory to work

File: src/robostilt_description/urdf/robostilt.urdf.xacro (robot description, xacro)
@@ -9,5 +9,5 @@
   <xacro:property name="limit_leg_upper" value="-0.1" />
   <xacro:property name="limit_leg_velocity" value="0.5" />
-  <xacro:property name="limit_leg_effort" value="2000.0" />
+  <xacro:property name="limit_leg_effort" value="1000.0" />
   <xacro:property name="limit_third_frame_prismatic_lower" value="${-1*frame_thickness}" />
   <xacro:property name="limit_third_frame_prismatic_upper" value="${-1*frame_length_x/3.0}" />

Commit message: Trajectory controller working

File: src/robostilt_description/urdf/robostilt.urdf.xacro (robot description, xacro)
@@ -20,9 +20,9 @@
 <!-- Friction and dynamics -->
 <xacro:macro name="friction" >
-      <mu1>0.3</mu1>
-      <mu2>0.3</mu2>
+      <mu1>0.6</mu1>
+      <mu2>0.6</mu2>
 </xacro:macro>
-  <xacro:property name="damping" value="0.7" />
-  <xacro:property name="damping_friction" value="0.3" />
+  <xacro:property name="damping" value="1.5" />
+  <xacro:property name="damping_friction" value="1.0" />
 <!-- MACROS -->
   <!-- Frames -->

Commit message: Step forward sequence working

File: src/robostilt_description/urdf/robostilt.urdf.xacro (robot description, xacro)
@@ -6,14 +6,14 @@
   <xacro:property name="frame_length_y" value="1.0" />
   <xacro:property name="frame_thickness" value="0.09" />
-  <xacro:property name="limit_leg_lower" value="-0.9" />
-  <xacro:property name="limit_leg_upper" value="-0.1" />
-  <xacro:property name="limit_leg_velocity" value="0.5" />
+  <xacro:property name="limit_leg_lower" value="-1.0" />
+  <xacro:property name="limit_leg_upper" value="0.0" />
+  <xacro:property name="limit_leg_velocity" value="1.0" />
   <xacro:property name="limit_leg_effort" value="1000.0" />
-  <xacro:property name="limit_third_frame_prismatic_lower" value="${-1*frame_thickness}" />
-  <xacro:property name="limit_third_frame_prismatic_upper" value="${-1*frame_length_x/3.0}" />
-  <xacro:property name="limit_third_frame_prismatic_velocity" value="0.5" />
-  <xacro:property name="limit_third_frame_prismatic_effort" value="1000.0" />
-  <xacro:property name="limit_third_frame_revolute_lower" value="-0.5" />
-  <xacro:property name="limit_third_frame_revolute_upper" value="0.5" />
+  <xacro:property name="limit_third_frame_prismatic_lower" value="-0.6" />
+  <xacro:property name="limit_third_frame_prismatic_upper" value="-0.2" />
+  <xacro:property name="limit_third_frame_prismatic_velocity" value="1.0" />
+  <xacro:property name="limit_third_frame_prismatic_effort" value="10000.0" />
+  <xacro:property name="limit_third_frame_revolute_lower" value="-0.3" />
+  <xacro:property name="limit_third_frame_revolute_upper" value="0.3" />
   <xacro:property name="limit_third_frame_revolute_velocity" value="0.5" />
   <xacro:property name="limit_third_frame_revolute_effort" value="1000.0" />
@@ -133,6 +133,6 @@
       </collision>
       <inertial>
-        <mass value="1.0" />
-        <inertia ixx="0.0001" ixy="0.0" ixz="0.0" iyy="0.0001" iyz="0.0" izz="0.0001" />
+        <mass value="0.1" />
+        <inertia ixx="0.001" ixy="0.0" ixz="0.0" iyy="0.001" iyz="0.0" izz="0.001" />
       </inertial>
   </link>

Commit message: URDF with arguments working

File: src/robostilt_description/urdf/robostilt.urdf.xacro (robot description, xacro)
@@ -2,20 +2,20 @@
 <robot name="robostilt" xmlns:xacro="http://www.ros.org/wiki/xacro" >  <!-- ROBOT NAME -->
 <!-- PROPERTIES -->
-  <xacro:property name="leg_length" value="1.0" />
-  <xacro:property name="frame_length_x" value="1.5" />
-  <xacro:property name="frame_length_y" value="1.0" />
-  <xacro:property name="frame_thickness" value="0.09" />
-  <xacro:property name="limit_leg_lower" value="-1.0" />
-  <xacro:property name="limit_leg_upper" value="0.0" />
-  <xacro:property name="limit_leg_velocity" value="1.0" />
-  <xacro:property name="limit_leg_effort" value="1000.0" />
-  <xacro:property name="limit_third_frame_prismatic_lower" value="-0.6" />
-  <xacro:property name="limit_third_frame_prismatic_upper" value="-0.2" />
-  <xacro:property name="limit_third_frame_prismatic_velocity" value="1.0" />
-  <xacro:property name="limit_third_frame_prismatic_effort" value="10000.0" />
-  <xacro:property name="limit_third_frame_revolute_lower" value="-0.3" />
-  <xacro:property name="limit_third_frame_revolute_upper" value="0.3" />
-  <xacro:property name="limit_third_frame_revolute_velocity" value="0.5" />
-  <xacro:property name="limit_third_frame_revolute_effort" value="1000.0" />
+  <xacro:property name="leg_length" value="$(arg leg_length)" />
+  <xacro:property name="frame_length_x" value="$(arg frame_length_x)" />
+  <xacro:property name="frame_length_y" value="$(arg frame_length_y)" />
+  <xacro:property name="frame_thickness" value="$(arg frame_thickness)" />
+  <xacro:property name="limit_leg_lower" value="$(arg limit_leg_lower)" />
+  <xacro:property name="limit_leg_upper" value="$(arg limit_leg_upper)" />
+  <xacro:property name="limit_leg_velocity" value="$(arg limit_leg_velocity)" />
+  <xacro:property name="limit_leg_effort" value="$(arg limit_leg_effort)" />
+  <xacro:property name="limit_third_frame_prismatic_lower" value="$(arg limit_third_frame_prismatic_lower)" />
+  <xacro:property name="limit_third_frame_prismatic_upper" value="$(arg limit_third_frame_prismatic_upper)" />
+  <xacro:property name="limit_third_frame_prismatic_velocity" value="$(arg limit_third_frame_prismatic_velocity)" />
+  <xacro:property name="limit_third_frame_prismatic_effort" value="$(arg limit_third_frame_prismatic_effort)" />
+  <xacro:property name="limit_third_frame_revolute_lower" value="$(arg limit_third_frame_revolute_lower)" />
+  <xacro:property name="limit_third_frame_revolute_upper" value="$(arg limit_third_frame_revolute_upper)" />
+  <xacro:property name="limit_third_frame_revolute_velocity" value="$(arg limit_third_frame_revolute_velocity)" />
+  <xacro:property name="limit_third_frame_revolute_effort" value="$(arg limit_third_frame_revolute_effort)" />
 <!-- Friction and dynamics -->
 <xacro:macro name="friction" >

Commit message: Gazebo offset model bug fixed

File: src/robostilt_description/urdf/robostilt.urdf.xacro (robot description, xacro)
@@ -50,6 +50,6 @@
         <geometry>
             <box size="${frame_thickness} ${frame_length_y-frame_thickness*1.1} ${frame_thickness}"/>
-          </geometry>
-          <origin rpy="0 0 0" xyz="${frame_length_x/2.0} 0 0"/>
+        </geometry>
+          <origin rpy="0 0 0" xyz="${-1*reflect*frame_length_x/2.0} 0 0"/>
         </collision>
         <inertial>
@@ -77,4 +77,5 @@
             <cylinder length="${leg_length}" radius="${frame_thickness/2.0}"/>
           </geometry>
+          <origin rpy="0 0 0" xyz="0.0 0.0 ${leg_length/2.0}"/>
         </collision>
         <inertial>
@@ -131,4 +132,5 @@
           <cylinder length="${frame_thickness}" radius="${frame_thickness/2.0}"/>
         </geometry>
+        <origin rpy="0 0 0" xyz="0.0 0.0 0.0"/>
       </collision>
       <inertial>

Commit message: Multiple joint controllers working

File: src/robostilt_description/urdf/robostilt.urdf.xacro (robot description, xacro)
@@ -27,5 +27,5 @@
 <!-- MACROS -->
   <!-- Frames -->
-   <xacro:macro name="frame_link" params="link_name material reflect" >
+   <xacro:macro name="frame" params="link_name material reflect" >
       <link name="${link_name}">
         <visual> <!-- X beam -->
@@ -84,5 +84,5 @@
         </inertial>
       </link>
-      <joint name="${parent}_to_leg_${suffix}" type="prismatic">
+      <joint name="leg_${suffix}" type="prismatic">
         <parent link="${parent}"/>
         <child link="leg_${suffix}"/>
@@ -96,10 +96,10 @@
         <xacro:gazebo_color material="${material}"/>
       </gazebo>
-      <transmission name="leg_${suffix}_trans">
+      <transmission name="leg_${suffix}">
         <type>transmission_interface/SimpleTransmission</type>
-        <joint name="${parent}_to_leg_${suffix}">
+        <joint name="leg_${suffix}">
           <hardwareInterface>hardware_interface/EffortJointInterface</hardwareInterface>
         </joint>
-        <actuator name="leg_${suffix}_motor">
+        <actuator name="leg_${suffix}">
           <hardwareInterface>hardware_interface/EffortJointInterface</hardwareInterface>
           <mechanicalReduction>1</mechanicalReduction>
@@ -119,5 +119,5 @@
 <!-- FRAMES -->
      <!-- Even frame -->
-  <xacro:frame_link link_name="base_link" material="Orange" reflect="1"/>
+  <xacro:frame link_name="base_link" material="Orange" reflect="1"/>
   <link name="third_frame"> <!-- Revolute joint -->
       <visual>
@@ -143,5 +143,5 @@
         <xacro:gazebo_color material="Yellow"/>
   </gazebo>
-  <joint name="base_link_to_third_frame" type="prismatic">
+  <joint name="third_frame_prismatic" type="prismatic">
       <parent link="base_link"/>
       <child link="third_frame"/>
@@ -151,10 +151,10 @@
        <dynamics damping="${damping}" friction="${damping_friction}" />
   </joint>
-  <transmission name="base_link_to_third_frame_trans">
+  <transmission name="third_frame_prismatic">
         <type>transmission_interface/SimpleTransmission</type>
-        <joint name="base_link_to_third_frame">
+        <joint name="third_frame_prismatic">
           <hardwareInterface>hardware_interface/EffortJointInterface</hardwareInterface>
         </joint>
-        <actuator name="third_frame_prismatic_motor">
+        <actuator name="third_frame_prismatic">
           <hardwareInterface>hardware_interface/EffortJointInterface</hardwareInterface>
           <mechanicalReduction>1</mechanicalReduction>
@@ -162,6 +162,6 @@
       </transmission>
    <!-- Odd frame -->
-   <xacro:frame_link link_name="odd_frame" material="Yellow" reflect="-1"/>
-  <joint name="third_frame_to_odd_frame" type="revolute">
+   <xacro:frame link_name="odd_frame" material="Yellow" reflect="-1"/>
+  <joint name="third_frame_revolute" type="revolute">
         <parent link="third_frame"/>
         <child link="odd_frame"/>
@@ -171,10 +171,10 @@
          <dynamics damping="${damping}" friction="${damping_friction}" />
   </joint>
-   <transmission name="third_frame_to_odd_frame_trans">
+   <transmission name="third_frame_revolute">
         <type>transmission_interface/SimpleTransmission</type>
-        <joint name="third_frame_to_odd_frame">
+        <joint name="third_frame_revolute">
           <hardwareInterface>hardware_interface/EffortJointInterface</hardwareInterface>
         </joint>
-        <actuator name="third_frame_revolute_motor">
+        <actuator name="third_frame_revolute">
           <hardwareInterface>hardware_interface/EffortJointInterface</hardwareInterface>
           <mechanicalReduction>1</mechanicalReduction>

Commit message: "Center of mass in progress"

File: src/robostilt_description/urdf/robostilt.urdf.xacro (robot description, xacro)
@@ -64,5 +64,5 @@
     </xacro:macro>
   <!-- Legs -->
-    <xacro:macro name="leg" params="suffix material parent x y">
+    <xacro:macro name="leg" params="suffix material parent x y z">
       <link name="leg_${suffix}">
         <visual>
@@ -89,5 +89,5 @@
         <limit effort="${limit_leg_effort}" lower="${limit_leg_lower}" upper="${limit_leg_upper}" velocity="${limit_leg_velocity}"/>
         <axis xyz="0 0 1"/>
-        <origin rpy="0 0 0" xyz="${x} ${y} 0.0"/>
+        <origin rpy="0 0 0" xyz="${x} ${y} ${z}"/>
         <dynamics damping="${damping}" friction="${damping_friction}" />
       </joint>
@@ -182,10 +182,10 @@
       </transmission>
 <!-- LEGS -->
- <xacro:leg suffix="1" material="Yellow" parent="odd_frame" x="${frame_length_x/2.0}" y="${frame_length_y/2.0}"/>
-  <xacro:leg suffix="3" material="Yellow" parent="odd_frame" x="${frame_length_x/2.0}" y="${-1*frame_length_y/2.0}"/>
-  <xacro:leg suffix="5" material="Yellow" parent="odd_frame" x="${-1*frame_length_x/2.0}" y="0"/>
-  <xacro:leg suffix="2" material="Orange" parent="base_link" x="${frame_length_x/2.0}" y="0"/>
-  <xacro:leg suffix="4" material="Orange" parent="base_link" x="${-1*frame_length_x/2.0}" y="${frame_length_y/2.0}"/>
-  <xacro:leg suffix="6" material="Orange" parent="base_link" x="${-1*frame_length_x/2.0} " y="${-1*frame_length_y/2.0}"/>
+ <xacro:leg suffix="1" material="Yellow" parent="odd_frame" x="${frame_length_x/2.0}" y="${frame_length_y/2.0}" z="${frame_thickness*-2.5}"/>
+  <xacro:leg suffix="3" material="Yellow" parent="odd_frame" x="${frame_length_x/2.0}" y="${-1*frame_length_y/2.0}" z="${frame_thickness*-2.5}"/>
+  <xacro:leg suffix="5" material="Yellow" parent="odd_frame" x="${-1*frame_length_x/2.0}" y="0" z="${frame_thickness*-2.5}"/>
+  <xacro:leg suffix="2" material="Orange" parent="base_link" x="${frame_length_x/2.0}" y="0" z="${frame_thickness/-2.0}"/>
+  <xacro:leg suffix="4" material="Orange" parent="base_link" x="${-1*frame_length_x/2.0}" y="${frame_length_y/2.0}" z="${frame_thickness/-2.0}"/>
+  <xacro:leg suffix="6" material="Orange" parent="base_link" x="${-1*frame_length_x/2.0} " y="${-1*frame_length_y/2.0}" z="${frame_thickness/-2.0}"/>
 <!-- GAZEBO -->
 <xacro:include filename="$(find robostilt_description)/urdf/robostilt.gazebo"/>

Commit message: CG marker displayed

File: src/robostilt_description/urdf/robostilt.urdf.xacro (robot description, xacro)
@@ -56,4 +56,5 @@
           <mass value="1.0" />
           <inertia ixx="0.008" ixy="0.0" ixz="0.0" iyy="0.08" iyz="0.0" izz="0.08" />
+          <origin rpy="0 0 0" xyz="${-1*reflect*frame_length_x/4.0} 0 0"/>
         </inertial>
       </link>
@@ -82,4 +83,5 @@
           <mass value="1.0" />
           <inertia ixx="0.08" ixy="0.0" ixz="0.0" iyy="0.08" iyz="0.0" izz="0.001" />
+          <origin rpy="0 0 0" xyz="0.0 0.0 0.0"/>
         </inertial>
       </link>
@@ -137,4 +139,5 @@
         <mass value="0.1" />
         <inertia ixx="0.001" ixy="0.0" ixz="0.0" iyy="0.001" iyz="0.0" izz="0.001" />
+        <origin rpy="0 0 0" xyz="0.0 0.0 0.0"/>
       </inertial>
   </link>

Commit message: laser scanner and object detection working

File: src/robostilt_description/urdf/robostilt.urdf.xacro (robot description, xacro)
@@ -193,3 +193,28 @@
 <!-- GAZEBO -->
 <xacro:include filename="$(find robostilt_description)/urdf/robostilt.gazebo"/>
+ <!--  Hokuyo Laser Sensor-->
+<link name="hokuyo_link">
+  <collision>
+    <origin xyz="0 0 0" rpy="0 0 0"/>
+    <geometry>
+      <cylinder length="0.1" radius="0.05"/>
+    </geometry>
+  </collision>
+  <visual>
+    <origin xyz="0 0 0" rpy="0 0 0"/>
+    <geometry>
+      <cylinder length="0.1" radius="0.05"/>
+    </geometry>
+  </visual>
+  <inertial>
+    <mass value="1e-5" />
+    <origin xyz="0 0 0" rpy="0 0 0"/>
+    <inertia ixx="1e-6" ixy="0" ixz="0" iyy="1e-6" iyz="0" izz="1e-6" />
+  </inertial>
+</link>
+<joint name="hokuyo_joint" type="fixed">
+  <origin xyz="${frame_length_x/2.0+0.1} 0.0 0.0" rpy="0 0 -0.0"/>
+  <parent link="base_link"/>
+  <child link="hokuyo_link"/>
+</joint>
 </robot>
