Commit message: Robot state received unkonwn fault

File: src/robostilt_description/urdf/materials.xacro (robot description, xacro)
@@ -5,5 +5,5 @@
   </material>
   <material name="Blue">
-    <color rgba="0.0 0.0 0.8 1.0"/>
+    <color rgba="0.0 0.0 1.0 1.0"/>
   </material>
   <material name="Green">

File: src/robostilt_description/urdf/robostilt.urdf.xacro (robot description, xacro)
@@ -128,5 +128,5 @@
         </geometry>
         <origin rpy="0 0 0" xyz="0.0 0.0 0.0"/>
-        <material name="Yellow"/>
+        <material name="Blue"/>
       </visual>
       <collision>
@@ -144,5 +144,5 @@
   <gazebo reference="third_frame">
          <xacro:friction/>
-        <xacro:gazebo_color material="Yellow"/>
+        <xacro:gazebo_color material="Blue"/>
   </gazebo>
   <joint name="third_frame_prismatic" type="prismatic">
